File: kicad/midi-biodata-v2.sch (KiCad schematic (older format))
At the start: 33 parts, among them J1 DIN-5_180degree, J2 Audio-Jack-2, J3 Conn_01x02, J4 Conn_01x02, SW1 SW_Push, U1 ATMEGA328P-AU, U2 POT_SWITCH, U3 LMC555xM, Y1 Crystal_GND2

Commit message: upload v2.1
Parts:
- removed R4: 0R, Resistors_SMD:R_0805, symbol R
- added C7: 100nF, Capacitors_SMD:C_0805, symbol C
- added C8: 1uF, Capacitors_SMD:C_0805, symbol C
- C1, C2, C3, C4: footprint Capacitors_SMD:C_0805 -> Capacitors_SMD:C_1206
- D8, D9: footprint Resistors_SMD:R_0805 -> Diodes_SMD:D_0805
- R1, R2, R3, R6, R7: footprint Resistors_SMD:R_0805 -> Resistors_SMD:R_1206
Connections:
- net GND: now also C7.1, C8.1
- net VCC: now also C7.2, C8.2
- net at U1.31 ((PCINT17/TXD)PD1): now also J1.5
- net at C3.2, D8.1 (A1), U3.2 (TR)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: now also J2.2; no longer J2.1
- net at D9.2 (A2), R6.2, U3.7 (DIS): now also J2.1; no longer J2.2
Changed lines of the file:
@@
 L Audio-Jack-2 J2
 U 1 1 5A2851FD
-P 6450 2100
-F 0 "J2" H 6425 2175 50  0000 C CNN
-F 1 "Audio-Jack-2" H 6425 1925 50  0000 C CNN
-F 2 "mono-jack:mono-jack" H 6700 2100 50  0001 C CNN
-F 3 "" H 6700 2100 50  0001 C CNN
-	1    6450 2100
-	-1   0    0    1
+P 6450 2000
+F 0 "J2" H 6425 2075 50  0000 C CNN
+F 1 "Audio-Jack-2" H 6425 1825 50  0000 C CNN
+F 2 "mono-jack:mono-jack" H 6700 2000 50  0001 C CNN
+F 3 "" H 6700 2000 50  0001 C CNN
+	1    6450 2000
+	-1   0    0    -1
 $EndComp
 $Comp
@@
 F 0 "C1" H 2575 3350 50  0000 L CNN
 F 1 "100nF" H 2575 3150 50  0000 L CNN
-F 2 "Capacitors_SMD:C_0805" H 2588 3100 50  0001 C CNN
+F 2 "Capacitors_SMD:C_1206" H 2588 3100 50  0001 C CNN
 F 3 "" H 2550 3250 50  0001 C CNN
 	1    2550 3250
@@
 F 0 "C3" H 4575 1800 50  0000 L CNN
 F 1 "4,7nF" H 4575 1600 50  0000 L CNN
-F 2 "Capacitors_SMD:C_0805" H 4588 1550 50  0001 C CNN
+F 2 "Capacitors_SMD:C_1206" H 4588 1550 50  0001 C CNN
 F 3 "" H 4550 1700 50  0001 C CNN
 	1    4550 1700
@@
 F 0 "C4" H 5375 1350 50  0000 L CNN
 F 1 "100nF" H 5375 1150 50  0000 L CNN
-F 2 "Capacitors_SMD:C_0805" H 5388 1100 50  0001 C CNN
+F 2 "Capacitors_SMD:C_1206" H 5388 1100 50  0001 C CNN
 F 3 "" H 5350 1250 50  0001 C CNN
 	1    5350 1250
@@
 F 0 "R6" V 6280 1550 50  0000 C CNN
 F 1 "100K" V 6200 1550 50  0000 C CNN
-F 2 "Resistors_SMD:R_0805" V 6130 1550 50  0001 C CNN
+F 2 "Resistors_SMD:R_1206" V 6130 1550 50  0001 C CNN
 F 3 "" H 6200 1550 50  0001 C CNN
 	1    6200 1550
@@
 L VCC #PWR07
 U 1 1 5A285FFB
-P 2250 3400
-F 0 "#PWR07" H 2250 3250 50  0001 C CNN
-F 1 "VCC" H 2250 3550 50  0000 C CNN
-F 2 "" H 2250 3400 50  0001 C CNN
-F 3 "" H 2250 3400 50  0001 C CNN
-	1    2250 3400
+P 2050 3400
+F 0 "#PWR07" H 2050 3250 50  0001 C CNN
+F 1 "VCC" H 2050 3550 50  0000 C CNN
+F 2 "" H 2050 3400 50  0001 C CNN
+F 3 "" H 2050 3400 50  0001 C CNN
+	1    2050 3400
 	1    0    0    -1
 $EndComp
@@
 F 0 "R1" V 4980 5300 50  0000 C CNN
 F 1 "220R" V 4900 5300 50  0000 C CNN
-F 2 "Resistors_SMD:R_0805" V 4830 5300 50  0001 C CNN
+F 2 "Resistors_SMD:R_1206" V 4830 5300 50  0001 C CNN
 F 3 "" H 4900 5300 50  0001 C CNN
 	1    4900 5300
@@
 F 0 "R2" V 5930 1550 50  0000 C CNN
 F 1 "220R" V 5850 1550 50  0000 C CNN
-F 2 "Resistors_SMD:R_0805" V 5780 1550 50  0001 C CNN
+F 2 "Resistors_SMD:R_1206" V 5780 1550 50  0001 C CNN
 F 3 "" H 5850 1550 50  0001 C CNN
 	1    5850 1550
@@
 F 0 "R3" V 6530 4900 50  0000 C CNN
 F 1 "220R" V 6450 4900 50  0000 C CNN
-F 2 "Resistors_SMD:R_0805" V 6380 4900 50  0001 C CNN
+F 2 "Resistors_SMD:R_1206" V 6380 4900 50  0001 C CNN
 F 3 "" H 6450 4900 50  0001 C CNN
 	1    6450 4900
@@
 F 0 "R7" V 6580 3700 50  0000 C CNN
 F 1 "3,9K" V 6500 3700 50  0000 C CNN
-F 2 "Resistors_SMD:R_0805" V 6430 3700 50  0001 C CNN
+F 2 "Resistors_SMD:R_1206" V 6430 3700 50  0001 C CNN
 F 3 "" H 6500 3700 50  0001 C CNN
 	1    6500 3700
@@
 F 0 "C2" H 6675 3950 50  0000 L CNN
 F 1 "100nF" H 6675 3750 50  0000 L CNN
-F 2 "Capacitors_SMD:C_0805" H 6688 3700 50  0001 C CNN
+F 2 "Capacitors_SMD:C_1206" H 6688 3700 50  0001 C CNN
 F 3 "" H 6650 3850 50  0001 C CNN
 	1    6650 3850
@@
 F 0 "D8" H 6200 2500 50  0000 C CNN
 F 1 "D_TVS" H 6200 2300 50  0000 C CNN
-F 2 "Resistors_SMD:R_0805" H 6200 2400 50  0001 C CNN
+F 2 "Diodes_SMD:D_0805" H 6200 2400 50  0001 C CNN
 F 3 "" H 6200 2400 50  0001 C CNN
 	1    6200 2400
@@
 F 0 "D9" H 6650 1700 50  0000 C CNN
 F 1 "D_TVS" H 6650 1500 50  0000 C CNN
-F 2 "Resistors_SMD:R_0805" H 6650 1600 50  0001 C CNN
+F 2 "Diodes_SMD:D_0805" H 6650 1600 50  0001 C CNN
 F 3 "" H 6650 1600 50  0001 C CNN
 	1    6650 1600
@@
 	4750 4250 5300 4250
 Wire Wire Line
-	2250 3400 2850 3400
+	2050 3400 2850 3400
 Wire Wire Line
 	5700 2050 5800 2050
@@
 	7400 5950 7650 5950
 Connection ~ 2850 3500
-$Comp
-L R R4
-U 1 1 5A528B6A
-P 5400 4900
-F 0 "R4" V 5480 4900 50  0000 C CNN
-F 1 "0R" V 5400 4900 50  0000 C CNN
-F 2 "Resistors_SMD:R_0805" V 5330 4900 50  0001 C CNN
-F 3 "" H 5400 4900 50  0001 C CNN
-	1    5400 4900
-	0    1    1    0
-$EndComp
-Wire Wire Line
-	5150 4900 5250 4900
-Wire Wire Line
-	5550 4900 5700 4900
+Wire Wire Line
+	5150 4900 5700 4900
 $Comp
 L C C6
@@
 	6200 1750 6650 1750
 Connection ~ 6200 1750
+$Comp
+L C C7
+U 1 1 5AA427EF
+P 2350 3250
+F 0 "C7" H 2375 3350 50  0000 L CNN
+F 1 "100nF" H 2375 3150 50  0000 L CNN
+F 2 "Capacitors_SMD:C_0805" H 2388 3100 50  0001 C CNN
+F 3 "" H 2350 3250 50  0001 C CNN
+	1    2350 3250
+	1    0    0    -1
+$EndComp
+$Comp
+L GND #PWR032
+U 1 1 5AA42881
+P 2350 3100
+F 0 "#PWR032" H 2350 2850 50  0001 C CNN
+F 1 "GND" H 2350 2950 50  0000 C CNN
+F 2 "" H 2350 3100 50  0001 C CNN
+F 3 "" H 2350 3100 50  0001 C CNN
+	1    2350 3100
+	0    1    1    0
+$EndComp
+Connection ~ 2350 3400
+$Comp
+L C C8
+U 1 1 5AA445D6
+P 2150 3250
+F 0 "C8" H 2175 3350 50  0000 L CNN
+F 1 "1uF" H 2175 3150 50  0000 L CNN
+F 2 "Capacitors_SMD:C_0805" H 2188 3100 50  0001 C CNN
+F 3 "" H 2150 3250 50  0001 C CNN
+	1    2150 3250
+	1    0    0    -1
+$EndComp
+$Comp
+L GND #PWR033
+U 1 1 5AA447C2
+P 2150 3100
+F 0 "#PWR033" H 2150 2850 50  0001 C CNN
+F 1 "GND" H 2150 2950 50  0000 C CNN
+F 2 "" H 2150 3100 50  0001 C CNN
+F 3 "" H 2150 3100 50  0001 C CNN
+	1    2150 3100
+	0    1    1    0
+$EndComp
+Connection ~ 2150 3400
 $EndSCHEMATC
